File: ptvo_fs.brd (EAGLE design)
At the start: 121.4 x 27.4 mm, 25 parts, among them U1 HTU21D

Commit message: Add files via upload
Parts:
- added C5, C6: 100nF, adafruit2:C0805
- added IC1: DS18S20USOP8, 1wire:UMAX8
- added R5: 2.2k, adafruit4:M0805
- added U$2: IS25LP080D, W25Q80BVSNIG:SO-8
- D1: value (none) -> PTSMD3528
- moved J2 1.80 mm to (24.1, 25.7)
- moved D1 0.81 mm to (33.6, 2.70)
- moved R3 0.73 mm to (39.0, 2.80)
- moved U1 0.70 mm to (2.90, 2.73), turned to 0 degrees
Connections:
- new net D9: U$1.DIO9, U$2.6
- net +3V3: now also C5.1, C6.1, IC1.8, R5.1, U$2.8
- net D07: now also R5.2, U$2.1
- net D08: now also U$2.2; no longer LED1.A
- net D10: now also U$2.5
- net D18: now also IC1.1
- net D25: now also LED1.A
- net GND: now also C5.2, C6.2, IC1.4, U$2.4
Routing:
- net +3V3: track 120.2 -> 141.8 mm
- net D18: track 6.04 -> 26.9 mm, vias 0 -> 2
- net D08: track 25.6 -> 9.62 mm, vias 0 -> 1
- net D07: track 0.00 -> 14.0 mm, vias 0 -> 1
- net D10: track 0.00 -> 11.7 mm, vias 0 -> 1
- net D25: track 6.03 -> 14.6 mm, vias 0 -> 1
- net D9: track 0.00 -> 8.27 mm, vias 0 -> 1
- net SCL: track 8.99 -> 4.65 mm
- net D27: track 56.5 -> 59.2 mm
- net D23: track 6.09 -> 4.25 mm
- net D24: track 6.02 -> 4.20 mm
- net D22: track 5.97 -> 4.15 mm
- net D16: track 6.01 -> 4.19 mm
- net D20: track 6.00 -> 4.18 mm
- net D21: track 6.04 -> 4.26 mm
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Other:
- board size 121.4 x 27.4 mm -> 121.4 x 25.5 mm
- board text added: "LED"

Commit message: Add files via upload
Parts:
- added Q1: SI2323DS, SI2323DS:SOT23
- moved R3 19.7 mm to (19.3, 2.70)
- moved D1 19.7 mm to (13.9, 2.70)
- moved C1 13.9 mm to (33.2, 23.6)
- moved C4 13.8 mm to (33.2, 19.8)
- moved SWITCH1 11.3 mm to (42.6, 24.5), turned to 0 degrees
- moved SWITCH 11.0 mm to (49.6, 24.5), turned to 0 degrees
- moved IC1 9.11 mm to (31.1, 3.10), turned to 90 degrees
- moved C5 5.00 mm to (31.1, 5.60)
Connections:
- new net N$5: BT1.+, Q1.3
- net +3V3: now also Q1.2; no longer BT1.+
- net GND: now also Q1.1
Routing:
- net D27: track 59.2 -> 36.8 mm
- net D11: track 19.5 -> 5.53 mm, vias 2 -> 0
- net D18: track 26.9 -> 37.6 mm
- net N$4: track 29.3 -> 38.2 mm
- net N$3: track 20.0 -> 28.6 mm
- net +3V3: track 141.8 -> 137.7 mm, vias 4 -> 7
- net N$5: track 0.00 -> 3.40 mm
- net GND: track 10.7 -> 11.4 mm, vias 121 -> 124

Commit message: Add files via upload
Parts:
- moved D1 3.50 mm to (10.4, 2.60)
- moved R3 3.50 mm to (15.8, 2.60)
- moved C4 2.60 mm to (35.8, 19.8)
- moved C3 1.10 mm to (6.17, 2.85), turned to 270 degrees
- moved TP2 0.10 mm to (52.0, 19.1)
Routing:
- net D27: track 36.8 -> 31.4 mm
- net D11: track 5.53 -> 9.19 mm
- net GND: track 11.4 -> 14.0 mm, vias 124 -> 132
- net +3V3: track 137.7 -> 136.5 mm

Commit message: Add files via upload
Parts:
- removed TP3, TP4, TP5, TP6, TP7, TP8: TPB1,27, testpad:B1,27
- added J1: (no value), SparkFun-Connectors2:1X05_1.27MM
- added U2: SHTC3, SHTC3:SON100P200X200X80-5N
- moved C6 1.30 mm to (9.70, 16.4)
- moved R5 1.30 mm to (14.1, 16.4)
- moved U$2 1.30 mm to (12.0, 13.1)
- moved U1 0.35 mm to (3.04, 3.04)
Connections:
- removed net N$4: SWITCH1.1, U$1.RES
- new net RST: J1.5, SWITCH1.1, U$1.RES
- net +3V3: now also J1.2, U2.1; no longer TP6.TP
- net GND: now also J1.1, U2.4, U2.5; no longer TP7.TP
- net RX: now also J1.3; no longer TP5.TP
- net SCL: now also U2.2
- net SDA: now also U2.3
- net TCK: now also J1.7; no longer TP8.TP
- net TMS: now also J1.6; no longer TP3.TP
- net TX: now also J1.4; no longer TP4.TP
Routing:
- net RST: track 0.00 -> 66.9 mm, vias 0 -> 4
- net N$4: track 38.2 -> 0.00 mm, vias 4 -> 0
- net GND: track 14.0 -> 20.4 mm, vias 132 -> 134
- net SCL: track 4.65 -> 9.01 mm, vias 0 -> 1
- net SDA: track 9.98 -> 14.2 mm, vias 0 -> 1
- net TX: track 33.3 -> 34.7 mm, vias 1 -> 0
- net D08: track 9.62 -> 10.9 mm
- net D07: track 14.0 -> 15.3 mm
- net D9: track 8.27 -> 9.45 mm
- net +3V3: track 136.5 -> 137.6 mm, vias 7 -> 6
- net RX: track 36.5 -> 37.5 mm, vias 1 -> 0
- net D10: track 11.7 -> 11.0 mm
- net D26: track 50.6 -> 50.1 mm
- net TMS: track 28.9 -> 29.2 mm, vias 1 -> 0
- net TCK: track 26.4 -> 26.5 mm, vias 1 -> 0
Other:
- board text added: "Firmware"
- board text added: "RST"
- board text added: "SBL"
- board text added: "TDI"
- board text added: "TDO"
- board text removed: "D15/SBL"
