File: ptvo_fs.sch (EAGLE design)
At the start: 25 parts, among them U1 HTU21D

Commit message: Add files via upload
Parts:
- added C5, C6: 100nF, adafruit2:C-USC0805
- added IC1: DS18S20USOP8, 1wire:DS18S20USOP8
- added R5: 2.2k, adafruit4:R-US_M0805
- added U$2: IS25LP080D, W25Q80BVSNIG:W25Q80BVSNIG
- D1: value (none) -> PTSMD3528
Connections:
- new net D9: U$1.DIO9, U$2.CLK
- net +3V3: now also C5.1, C6.1, IC1.VDD, R5.1, U$2.VCC
- net D07: now also R5.2, U$2.CS
- net D08: now also U$2.DO/IO1; no longer LED1.A
- net D10: now also U$2.DI/IO0
- net D18: now also IC1.DQ
- net D25: now also LED1.A
- net GND: now also C5.2, C6.2, IC1.GND, U$2.GND
Changed lines of the file:
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@@
 <part name="GND2" library="supply1" library_urn="urn:adsk.eagle:library:371" deviceset="GND" device=""/>
 <part name="+3V1" library="supply1" library_urn="urn:adsk.eagle:library:371" deviceset="+3V3" device="" value="+3V"/>
-<part name="D1" library="diode" library_urn="urn:adsk.eagle:library:210" deviceset="DIODE-" device="DO214BA" package3d_urn="urn:adsk.eagle:package:43453/2"/>
+<part name="D1" library="diode" library_urn="urn:adsk.eagle:library:210" deviceset="DIODE-" device="DO214BA" package3d_urn="urn:adsk.eagle:package:43453/2" value="PTSMD3528"/>
 <part name="R3" library="adafruit4" deviceset="R-US_" device="M0805" package3d_urn="urn:adsk.eagle:package:6240587/1" value="10k"/>
 <part name="GND3" library="supply1" library_urn="urn:adsk.eagle:library:371" deviceset="GND" device=""/>
@@
 <part name="SWITCH1" library="SPST Round Button" deviceset="SKRKAEE010" device=""/>
 <part name="GND9" library="supply1" library_urn="urn:adsk.eagle:library:371" deviceset="GND" device=""/>
+<part name="U$2" library="W25Q80BVSNIG" deviceset="W25Q80BVSNIG" device="" value="IS25LP080D"/>
+<part name="GND10" library="supply1" library_urn="urn:adsk.eagle:library:371" deviceset="GND" device=""/>
+<part name="GND24" library="supply1" library_urn="urn:adsk.eagle:library:371" deviceset="GND" device=""/>
+<part name="R5" library="adafruit4" deviceset="R-US_" device="M0805" package3d_urn="urn:adsk.eagle:package:6240587/1" value="2.2k"/>
+<part name="+3V6" library="supply1" library_urn="urn:adsk.eagle:library:371" deviceset="+3V3" device="" value="+3V"/>
+<part name="+3V7" library="supply1" library_urn="urn:adsk.eagle:library:371" deviceset="+3V3" device="" value="+3V"/>
+<part name="C6" library="adafruit2" deviceset="C-US" device="C0805" package3d_urn="urn:adsk.eagle:package:6240337/1" value="100nF"/>
+<part name="IC1" library="1wire" deviceset="DS18S20" device="USOP8"/>
+<part name="+3V8" library="supply1" library_urn="urn:adsk.eagle:library:371" deviceset="+3V3" device="" value="+3V"/>
+<part name="GND11" library="supply1" library_urn="urn:adsk.eagle:library:371" deviceset="GND" device=""/>
+<part name="C5" library="adafruit2" deviceset="C-US" device="C0805" package3d_urn="urn:adsk.eagle:package:6240337/1" value="100nF"/>
+<part name="GND12" library="supply1" library_urn="urn:adsk.eagle:library:371" deviceset="GND" device=""/>
 </parts>
 <sheets>
@@
 <instance part="D1" gate="G$1" x="63.5" y="43.18" smashed="yes" rot="R90">
 <attribute name="NAME" x="63.0174" y="45.72" size="1.778" layer="95" rot="R90"/>
-<attribute name="VALUE" x="65.8114" y="45.72" size="1.778" layer="96" rot="R90"/>
 </instance>
 <instance part="R3" gate="G$1" x="63.5" y="33.02" smashed="yes" rot="R90">
@@
 <instance part="GND9" gate="1" x="78.74" y="7.62" smashed="yes">
 <attribute name="VALUE" x="76.2" y="5.08" size="1.778" layer="96"/>
+</instance>
+<instance part="U$2" gate="G$1" x="261.62" y="43.18" smashed="yes"/>
+<instance part="GND10" gate="1" x="238.76" y="25.4" smashed="yes">
+<attribute name="VALUE" x="236.22" y="22.86" size="1.778" layer="96"/>
+</instance>
+<instance part="GND24" gate="1" x="284.48" y="53.34" smashed="yes" rot="R180">
+<attribute name="VALUE" x="287.02" y="55.88" size="1.778" layer="96" rot="R180"/>
+</instance>
+<instance part="R5" gate="G$1" x="289.56" y="40.64" smashed="yes" rot="R180">
+<attribute name="NAME" x="289.56" y="39.116" size="1.778" layer="95" font="vector" rot="R180" align="bottom-center"/>
+</instance>
+<instance part="+3V6" gate="G$1" x="302.26" y="40.64" smashed="yes" rot="R270">
+<attribute name="VALUE" x="294.64" y="40.64" size="1.778" layer="96"/>
+</instance>
+<instance part="+3V7" gate="G$1" x="233.68" y="40.64" smashed="yes" rot="R90">
+<attribute name="VALUE" x="236.22" y="40.64" size="1.778" layer="96"/>
+</instance>
+<instance part="C6" gate="G$1" x="238.76" y="35.56" smashed="yes">
+<attribute name="NAME" x="239.776" y="36.195" size="1.778" layer="95"/>
+<attribute name="VALUE" x="239.776" y="31.369" size="1.778" layer="96"/>
+</instance>
+<instance part="IC1" gate="G$1" x="264.16" y="12.7" smashed="yes"/>
+<instance part="+3V8" gate="G$1" x="279.4" y="25.4" smashed="yes">
+<attribute name="VALUE" x="279.4" y="25.4" size="1.778" layer="96"/>
+</instance>
+<instance part="GND11" gate="1" x="246.38" y="7.62" smashed="yes">
+<attribute name="VALUE" x="243.84" y="5.08" size="1.778" layer="96"/>
+</instance>
+<instance part="C5" gate="G$1" x="279.4" y="15.24" smashed="yes">
+<attribute name="NAME" x="280.416" y="15.875" size="1.778" layer="95"/>
+<attribute name="VALUE" x="280.416" y="11.049" size="1.778" layer="96"/>
+</instance>
+<instance part="GND12" gate="1" x="279.4" y="5.08" smashed="yes">
+<attribute name="VALUE" x="276.86" y="2.54" size="1.778" layer="96"/>
 </instance>
 </instances>
@@
 <pinref part="GND9" gate="1" pin="GND"/>
 </segment>
+<segment>
+<pinref part="U$2" gate="G$1" pin="GND"/>
+<wire x1="279.4" y1="48.26" x2="284.48" y2="48.26" width="0.1524" layer="91"/>
+<pinref part="GND24" gate="1" pin="GND"/>
+<wire x1="284.48" y1="48.26" x2="284.48" y2="50.8" width="0.1524" layer="91"/>
+</segment>
+<segment>
+<pinref part="GND10" gate="1" pin="GND"/>
+<pinref part="C6" gate="G$1" pin="2"/>
+<wire x1="238.76" y1="27.94" x2="238.76" y2="30.48" width="0.1524" layer="91"/>
+</segment>
+<segment>
+<pinref part="IC1" gate="G$1" pin="GND"/>
+<wire x1="251.46" y1="12.7" x2="246.38" y2="12.7" width="0.1524" layer="91"/>
+<wire x1="246.38" y1="12.7" x2="246.38" y2="10.16" width="0.1524" layer="91"/>
+<pinref part="GND11" gate="1" pin="GND"/>
+</segment>
+<segment>
+<pinref part="C5" gate="G$1" pin="2"/>
+<wire x1="279.4" y1="10.16" x2="279.4" y2="7.62" width="0.1524" layer="91"/>
+<pinref part="GND12" gate="1" pin="GND"/>
+</segment>
 </net>
 <net name="D14" class="0">
@@
 <wire x1="208.28" y1="43.18" x2="215.9" y2="43.18" width="0.1524" layer="91"/>
 </segment>
+<segment>
+<pinref part="R5" gate="G$1" pin="1"/>
+<wire x1="294.64" y1="40.64" x2="299.72" y2="40.64" width="0.1524" layer="91"/>
+<pinref part="+3V6" gate="G$1" pin="+3V3"/>
+</segment>
+<segment>
+<pinref part="U$2" gate="G$1" pin="VCC"/>
+<wire x1="236.22" y1="40.64" x2="238.76" y2="40.64" width="0.1524" layer="91"/>
+<pinref part="+3V7" gate="G$1" pin="+3V3"/>
+<pinref part="C6" gate="G$1" pin="1"/>
+<wire x1="238.76" y1="40.64" x2="243.84" y2="40.64" width="0.1524" layer="91"/>
+<wire x1="238.76" y1="40.64" x2="238.76" y2="38.1" width="0.1524" layer="91"/>
+<junction x="238.76" y="40.64"/>
+</segment>
+<segment>
+<pinref part="IC1" gate="G$1" pin="VDD"/>
+<wire x1="276.86" y1="20.32" x2="279.4" y2="20.32" width="0.1524" layer="91"/>
+<wire x1="279.4" y1="20.32" x2="279.4" y2="22.86" width="0.1524" layer="91"/>
+<pinref part="+3V8" gate="G$1" pin="+3V3"/>
+<pinref part="C5" gate="G$1" pin="1"/>
+<wire x1="279.4" y1="20.32" x2="279.4" y2="17.78" width="0.1524" layer="91"/>
+<junction x="279.4" y="20.32"/>
+</segment>
 </net>
 <net name="D07" class="0">
@@
 <label x="106.68" y="33.02" size="1.778" layer="95"/>
 </segment>
+<segment>
+<pinref part="U$2" gate="G$1" pin="CS"/>
+<wire x1="279.4" y1="40.64" x2="284.48" y2="40.64" width="0.1524" layer="91"/>
+<pinref part="R5" gate="G$1" pin="2"/>
+<label x="279.4" y="40.64" size="1.778" layer="95"/>
+</segment>
 </net>
 <net name="D11" class="0">
@@
 <net name="D08" class="0">
 <segment>
-<pinref part="LED1" gate="G$1" pin="A"/>
-<wire x1="53.34" y1="45.72" x2="53.34" y2="53.34" width="0.1524" layer="91"/>
-<label x="53.34" y="53.34" size="1.778" layer="95" rot="R270"/>
-</segment>
-<segment>
 <pinref part="U$1" gate="G$1" pin="DIO8"/>
 <wire x1="116.84" y1="30.48" x2="106.68" y2="30.48" width="0.1524" layer="91"/>
 <label x="106.68" y="30.48" size="1.778" layer="95"/>
 </segment>
+<segment>
+<pinref part="U$2" gate="G$1" pin="DO/IO1"/>
+<wire x1="279.4" y1="43.18" x2="284.48" y2="43.18" width="0.1524" layer="91"/>
+<label x="279.4" y="43.18" size="1.778" layer="95"/>
+</segment>
 </net>
 <net name="D10" class="0">
@@
 <wire x1="116.84" y1="25.4" x2="106.68" y2="25.4" width="0.1524" layer="91"/>
 <label x="106.68" y="25.4" size="1.778" layer="95"/>
+</segment>
+<segment>
+<pinref part="U$2" gate="G$1" pin="DI/IO0"/>
+<wire x1="243.84" y1="48.26" x2="236.22" y2="48.26" width="0.1524" layer="91"/>
+<label x="236.22" y="48.26" size="1.778" layer="95"/>
 </segment>
 </net>
@@
 <label x="210.82" y="17.78" size="1.778" layer="95"/>
 </segment>
+<segment>
+<pinref part="LED1" gate="G$1" pin="A"/>
+<wire x1="53.34" y1="45.72" x2="53.34" y2="53.34" width="0.1524" layer="91"/>
+<label x="53.34" y="48.26" size="1.778" layer="95" rot="R90"/>
+</segment>
 </net>
 <net name="D24" class="0">
@@
 <label x="210.82" y="35.56" size="1.778" layer="95"/>
 </segment>
+<segment>
+<pinref part="IC1" gate="G$1" pin="DQ"/>
+<wire x1="251.46" y1="20.32" x2="246.38" y2="20.32" width="0.1524" layer="91"/>
+<label x="246.38" y="20.32" size="1.778" layer="95"/>
+</segment>
 </net>
 <net name="D17" class="0">
@@
 </segment>
 </net>
+<net name="D9" class="0">
+<segment>
+<pinref part="U$2" gate="G$1" pin="CLK"/>
+<wire x1="243.84" y1="45.72" x2="236.22" y2="45.72" width="0.1524" layer="91"/>
+<label x="236.22" y="45.72" size="1.778" layer="95"/>
+</segment>
+<segment>
+<pinref part="U$1" gate="G$1" pin="DIO9"/>
+<wire x1="116.84" y1="27.94" x2="106.68" y2="27.94" width="0.1524" layer="91"/>
+<label x="106.68" y="27.94" size="1.778" layer="95"/>
+</segment>
+</net>

Commit message: Add files via upload
Parts:
- added Q1: SI2323DS, SI2323DS:SI2323DS
Connections:
- new net N$5: BT1.+, Q1.D
- net +3V3: now also Q1.S; no longer BT1.+
- net GND: now also Q1.G
Other:
- moved on the sheet: BT1, C1, C2, C3, C4, C5, C6, D1, D5, LED1, R1, R2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

Commit message: Add files via upload
Other:
- moved on the sheet: BT1, C1, C2, C3, C4, C5, C6, D1, D5, LED1, Q1, R1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

Commit message: Add files via upload
Parts:
- removed TP3, TP4, TP5, TP6, TP7, TP8: TPB1,27, testpad:TPB1,27
- added J1: (no value), SparkFun-Connectors2:CONN_051.27MM
- added U2: SHTC3, SHTC3:SHTC3
Connections:
- removed net N$4: SWITCH1.1, U$1.RES
- new net RST: J1.5, SWITCH1.1, U$1.RES
- net +3V3: now also J1.2, U2.VDD; no longer TP6.TP
- net GND: now also J1.1, U2.EXP, U2.VSS; no longer TP7.TP
- net RX: now also J1.3; no longer TP5.TP
- net SCL: now also U2.SCL
- net SDA: now also U2.SDA
- net TCK: now also J1.7; no longer TP8.TP
- net TMS: now also J1.6; no longer TP3.TP
- net TX: now also J1.4; no longer TP4.TP
Other:
- moved on the sheet: BT1, C1, C2, C3, C4, C5, C6, D1, D5, LED1, Q1, R1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
