File: CC2652RB/ptvo_fs.brd (EAGLE design)
At the start: 100 x 25.5 mm, 30 parts, among them IC1 DS18S20USOP8, Q1 SI2323DS, U1 SHTC3, U2 E72-2G4M05S1F, Y1 Q22FA12800150

Commit message: Add files via upload
Parts:
- added IC2: BME280, bosch-bme280:BME280
Connections:
- net +3V3: now also IC2.2, IC2.6, IC2.8
- net GND: now also IC2.1, IC2.5, IC2.7
- net SCL: now also IC2.4
- net SDA: now also IC2.3
Routing:
- net SDA: track 2.78 -> 12.1 mm, vias 0 -> 1
- net GND: track 19.0 -> 26.4 mm, vias 36 -> 37
- net +3V3: track 62.3 -> 69.2 mm, vias 4 -> 5
- net SCL: track 2.49 -> 9.24 mm, vias 0 -> 1
Changed lines of the file:
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@@
 <attribute name="NAME" x="2.389" y="16.535" size="0.8128" layer="26" font="vector" rot="MR0"/>
 </element>
+<element name="IC2" library="bosch-bme280" package="BME280" value="BME280" x="2.9" y="2.6" smashed="yes" rot="MR270"/>
 </elements>
 <signals>
@@
 <wire x1="2.4" y1="1.5" x2="2.5" y2="1.4" width="0.2032" layer="1"/>
 <wire x1="2.5" y1="1.4" x2="2.6" y2="1.5" width="0.2032" layer="1"/>
-<wire x1="2.6" y1="1.5" x2="2.6" y2="2" width="0.2032" layer="1"/>
+<wire x1="2.6" y1="1.5" x2="2.6" y2="1.6" width="0.2032" layer="1"/>
 <polygon width="0.2032" layer="16" thermals="no">
-<vertex x="0.6" y="4.1"/>
-<vertex x="5" y="4.1"/>
+<vertex x="0.6" y="4.6"/>
+<vertex x="5" y="4.6"/>
 <vertex x="5" y="0"/>
 <vertex x="31.3" y="0"/>
@@
 </polygon>
 <polygon width="0.2032" layer="1" thermals="no">
-<vertex x="0.7" y="4.1"/>
-<vertex x="5" y="4.1"/>
+<vertex x="0.7" y="4.6"/>
+<vertex x="5" y="4.6"/>
 <vertex x="5" y="-0.4"/>
 <vertex x="31.3" y="-0.4"/>
@@
 <vertex x="0.7" y="26"/>
 </polygon>
-<via x="2.6" y="2" extent="1-16" drill="0.2"/>
-<wire x1="2.6" y1="2" x2="2.6" y2="3" width="0.1524" layer="16"/>
-<wire x1="2.6" y1="3" x2="3.1" y2="3.5" width="0.1524" layer="16"/>
-<wire x1="3.1" y1="3.5" x2="3.1" y2="4.2" width="0.1524" layer="16"/>
+<via x="2.6" y="1.6" extent="1-16" drill="0.2"/>
 <via x="25.6" y="14.8" extent="1-16" drill="0.25"/>
 <via x="25.6" y="16.1" extent="1-16" drill="0.25"/>
@@
 <via x="28.8" y="1.2" extent="1-16" drill="0.25"/>
 <via x="30.7" y="17.8" extent="1-16" drill="0.25"/>
+<contactref element="IC2" pad="7"/>
+<contactref element="IC2" pad="1"/>
+<contactref element="IC2" pad="5"/>
+<wire x1="2.6" y1="1.6" x2="2.7" y2="1.7" width="0.2" layer="16"/>
+<wire x1="2.7" y1="3.1" x2="2.7" y2="1.7" width="0.2" layer="16"/>
+<wire x1="3.2" y1="4.8" x2="3.2" y2="3.6" width="0.2" layer="16"/>
+<wire x1="2.7" y1="3.1" x2="3.2" y2="3.6" width="0.2" layer="16"/>
+<wire x1="1.875" y1="2.275" x2="1.335" y2="2.275" width="0.2" layer="16"/>
+<wire x1="1.335" y1="2.275" x2="1.21" y2="2.4" width="0.2" layer="16"/>
+<wire x1="1.21" y1="2.4" x2="1.21" y2="3.41" width="0.2" layer="16"/>
+<wire x1="1.375" y1="3.575" x2="1.875" y2="3.575" width="0.2" layer="16"/>
+<wire x1="1.21" y1="3.41" x2="1.375" y2="3.575" width="0.2" layer="16"/>
+<wire x1="1.875" y1="3.575" x2="1.875" y2="4.675" width="0.2" layer="16"/>
+<wire x1="1.875" y1="4.675" x2="2" y2="4.8" width="0.2" layer="16"/>
+<wire x1="2" y1="4.8" x2="3.2" y2="4.8" width="0.2" layer="16"/>
+<wire x1="2.6" y1="1.6" x2="2.625" y2="1.625" width="0.2" layer="16"/>
+<wire x1="2.625" y1="1.625" x2="3.925" y2="1.625" width="0.2" layer="16"/>
+<wire x1="2.6" y1="2" x2="2.6" y2="1.5" width="0.2" layer="1"/>
+<via x="5.2" y="3" extent="1-16" drill="0.25"/>
 <wire x1="7.625" y1="24.625" x2="7.6" y2="24.95" width="0" layer="19" extent="1-16"/>
 </signal>
@@
 <contactref element="U1" pad="1"/>
 <contactref element="C3" pad="1"/>
-<wire x1="3.57" y1="1.5" x2="5.575" y2="1.5" width="0.2032" layer="1"/>
+<wire x1="3.57" y1="1.5" x2="4.6" y2="1.5" width="0.2032" layer="1"/>
+<wire x1="4.6" y1="1.5" x2="5.575" y2="1.5" width="0.2032" layer="1"/>
 <wire x1="5.575" y1="1.5" x2="5.725" y2="1.65" width="0.2032" layer="1"/>
 <wire x1="17.075" y1="16.39" x2="19.54" y2="16.39" width="0.6096" layer="1"/>
@@
 <wire x1="22.5" y1="6.1" x2="22.7" y2="6.3" width="0.254" layer="16"/>
 <wire x1="20.679675" y1="6.1" x2="22.5" y2="6.1" width="0.254" layer="16"/>
+<contactref element="IC2" pad="6"/>
+<contactref element="IC2" pad="2"/>
+<contactref element="IC2" pad="8"/>
+<wire x1="2.352" y1="2.544025" x2="2.352" y2="2.005975" width="0.2" layer="16"/>
+<wire x1="2.352" y1="2.005975" x2="1.971025" y2="1.625" width="0.2" layer="16"/>
+<wire x1="1.875" y1="1.625" x2="1.971025" y2="1.625" width="0.2" layer="16"/>
+<wire x1="2.352" y1="2.544025" x2="1.971025" y2="2.925" width="0.2" layer="16"/>
+<wire x1="1.875" y1="2.925" x2="1.971025" y2="2.925" width="0.2" layer="16"/>
+<via x="4.6" y="1.5" extent="1-16" drill="0.25"/>
+<wire x1="3.925" y1="2.275" x2="4.425" y2="2.275" width="0.2" layer="16"/>
+<wire x1="4.425" y1="2.275" x2="4.6" y2="2.1" width="0.2" layer="16"/>
+<wire x1="4.6" y1="2.1" x2="4.6" y2="1.5" width="0.2" layer="16"/>
+<wire x1="1.875" y1="1.625" x2="1.875" y2="1.225" width="0.2" layer="16"/>
+<wire x1="1.875" y1="1.225" x2="2.2" y2="0.9" width="0.2" layer="16"/>
+<wire x1="4.6" y1="1.1" x2="4.6" y2="1.5" width="0.2" layer="16"/>
+<wire x1="2.2" y1="0.9" x2="4.4" y2="0.9" width="0.2" layer="16"/>
+<wire x1="4.4" y1="0.9" x2="4.6" y2="1.1" width="0.2" layer="16"/>
 </signal>
 <signal name="D11">
@@
 <wire x1="3.5" y1="3" x2="3.5" y2="2.57" width="0.2" layer="1"/>
 <wire x1="3.5" y1="2.57" x2="3.57" y2="2.5" width="0.2" layer="1"/>
+<contactref element="IC2" pad="4"/>
+<via x="2.4" y="6.8" extent="1-16" drill="0.25"/>
+<wire x1="3.725" y1="6.175" x2="3.725" y2="4.87" width="0.2" layer="1"/>
+<wire x1="3.9" y1="3.6" x2="3.9" y2="4.8" width="0.2" layer="16"/>
+<wire x1="3.925" y1="3.575" x2="3.9" y2="3.6" width="0.2" layer="16"/>
+<wire x1="2.4" y1="6.3" x2="2.4" y2="6.8" width="0.2" layer="16"/>
+<wire x1="3.9" y1="4.8" x2="2.4" y2="6.3" width="0.2" layer="16"/>
+<wire x1="3.1" y1="6.8" x2="2.4" y2="6.8" width="0.2" layer="1"/>
+<wire x1="3.725" y1="6.175" x2="3.1" y2="6.8" width="0.2" layer="1"/>
 </signal>
 <signal name="SDA">
@@
 <wire x1="2.625" y1="3.825" x2="2.625" y2="4.87" width="0.2" layer="1"/>
 <wire x1="1.63" y1="2.83" x2="2.625" y2="3.825" width="0.2" layer="1"/>
+<contactref element="IC2" pad="3"/>
+<wire x1="3.925" y1="2.925" x2="4.325" y2="2.925" width="0.2" layer="16"/>
+<wire x1="4.325" y1="2.925" x2="4.5" y2="3.1" width="0.2" layer="16"/>
+<wire x1="4.5" y1="3.1" x2="4.5" y2="4.7" width="0.2" layer="16"/>
+<wire x1="2.9" y1="6.3" x2="2.9" y2="7" width="0.2" layer="16"/>
+<wire x1="2.9" y1="7" x2="2.4" y2="7.5" width="0.2" layer="16"/>
+<wire x1="4.5" y1="4.7" x2="2.9" y2="6.3" width="0.2" layer="16"/>
+<via x="2.4" y="7.5" extent="1-16" drill="0.25"/>
+<wire x1="2.4" y1="7.5" x2="2.1" y2="7.5" width="0.2" layer="1"/>
+<wire x1="2.1" y1="7.5" x2="1.8536" y2="7.2536" width="0.2" layer="1"/>
+<wire x1="2.625" y1="5.875" x2="2.625" y2="4.87" width="0.2" layer="1"/>
+<wire x1="1.8536" y1="7.2536" x2="1.8536" y2="6.6464" width="0.2" layer="1"/>
+<wire x1="1.8536" y1="6.6464" x2="2.625" y2="5.875" width="0.2" layer="1"/>
 </signal>
 <signal name="N$3">
@@
 </drawing>
 <compatibility>
+<note version="6.3" minversion="6.2.2" severity="warning">
+Since Version 6.2.2 text objects can contain more than one line,
+which will not be processed correctly with this version.
+</note>
 <note version="8.2" severity="warning">
 Since Version 8.2, EAGLE supports online libraries. The ids

Commit message: Add files via upload
Parts:
- moved SWITCH 3.72 mm to (25.3, 22.7), turned to 270 degrees
- moved TP1 2.90 mm to (27.8, 13.8)
- moved R1 2.80 mm to (26.8, 13.8)
- moved D5 2.70 mm to (26.7, 11.7)
- moved TP2 2.20 mm to (28.8, 18.5)
- moved SWITCH1 1.55 mm to (21.8, 22.7), turned to 270 degrees
- moved D1 1.10 mm to (12.6, 1.90)
- moved Q1 0.91 mm to (26.3, 2.50)
- moved R3 0.81 mm to (17.8, 2.70)
- moved C1 0.71 mm to (21.6, 5.60)
- moved C2 0.60 mm to (25.5, 7.83)
- moved R2 0.60 mm to (27.6, 7.83)
Routing:
- net N$1: track 7.80 -> 19.1 mm
- net D24: track 18.6 -> 15.7 mm
- net GND: track 26.4 -> 29.2 mm, vias 37 -> 33
- net N$3: track 29.0 -> 31.3 mm
- net RST: track 20.3 -> 18.5 mm
- net D23: track 21.2 -> 19.9 mm
- net D11: track 4.48 -> 5.64 mm
- net N$4: track 30.9 -> 30.1 mm
- net D25: track 23.7 -> 23.6 mm, vias 1 -> 0

Commit message: Add files via upload
Parts:
- removed D1: PTSMD3528, diode:DO214BA
- added C7: 100nF, discretes-dev:CAPC1005X40N
- added R5: 4.7k, RC0402FR-073M6L:RESC1005X40N
- added U3: BH1750FVI-TR, BH1750FVI-TR:XDCR_BH1750FVI-TR
- R3: value 10k -> 4.7k; device adafruit4:M0805 -> RC0402FR-073M6L:RESC1005X40N
- moved R3 6.25 mm to (11.6, 2.00), turned to 90 degrees
- moved SWITCH 3.72 mm to (28.7, 24.2), turned to 0 degrees
- moved TP1 2.90 mm to (30.7, 13.8)
- moved R1 2.80 mm to (29.6, 13.8)
- moved D5 2.70 mm to (29.4, 11.8)
- moved TP2 2.20 mm to (30.9, 18.5)
- moved SWITCH1 1.55 mm to (22.2, 24.2), turned to 0 degrees
- moved Q1 0.91 mm to (27.2, 2.60)
- moved C1 0.71 mm to (22.3, 5.70)
- moved C2 0.60 mm to (26.1, 7.83)
- moved R2 0.60 mm to (28.1, 7.83)
Connections:
- new net N$6: C7.1, R3.2, U3.5
- new net N$9: R5.1, U3.2
- net +3V3: now also R3.1, U3.1
- net D11: no longer D1.C
- net D25: no longer D1.A, R3.2
- net GND: now also C7.2, R5.2, U3.3; no longer R3.1
- net SCL: now also U3.6
- net SDA: now also U3.4
Routing:
- net D25: track 23.6 -> 0.00 mm
- net SCL: track 9.24 -> 32.4 mm, vias 1 -> 2
- net SDA: track 12.1 -> 31.9 mm
- net +3V3: track 69.5 -> 76.2 mm, vias 5 -> 6
- net N$3: track 31.3 -> 37.5 mm
- net D11: track 5.64 -> 0.00 mm
- net N$1: track 19.1 -> 15.3 mm
- net D24: track 15.7 -> 18.6 mm
- net N$6: track 0.00 -> 2.88 mm
- net GND: track 29.2 -> 26.4 mm, vias 33 -> 41
- net N$9: track 0.00 -> 1.97 mm
- net RST: track 18.5 -> 20.3 mm
- net D23: track 19.9 -> 21.2 mm
- net N$4: track 30.1 -> 30.9 mm
