File: CC2652RB/ptvo_fs.sch (EAGLE design)
At the start: 30 parts, among them IC1 DS18S20USOP8, Q1 SI2323DS, U1 SHTC3, U2 E72-2G4M05S1F, Y1 Q22FA12800150

Commit message: Add files via upload
Parts:
- added IC2: BME280, bosch-bme280:BME280
Connections:
- net +3V3: now also IC2.CSB, IC2.VDD, IC2.VDDIO
- net GND: now also IC2.GND, IC2.SDO
- net SCL: now also IC2.SCK
- net SDA: now also IC2.SDI
Other:
- moved on the sheet: C6, C9, SWITCH, SWITCH1, U2, Y1

Commit message: Add files via upload
Parts:
- removed D1: PTSMD3528, diode:DIODE-DO214BA
- added C7: 100nF, discretes-dev:CAP0402
- added R5: 4.7k, RC0402FR-073M6L:RC0402FR-073M6L
- added U3: BH1750FVI-TR, BH1750FVI-TR:BH1750FVI-TR
- R3: value 10k -> 4.7k; device adafruit4:R-US_M0805 -> RC0402FR-073M6L:RC0402FR-073M6L
Connections:
- new net N$6: C7.1, R3.2, U3.DVI
- new net N$9: R5.1, U3.ADDR
- net +3V3: now also R3.1, U3.VCC
- net D11: no longer D1.C
- net D25: no longer D1.A, R3.2
- net GND: now also C7.2, R5.2, U3.GND; no longer R3.1
- net SCL: now also U3.SCL
- net SDA: now also U3.SDA
Other:
- moved on the sheet: BT1, C1, C2, C4, C5, D5, LED1, Q1, R1, R2, R3, R4
